File: board/DDT_i2c_proto_breakboard.kicad_sch (KiCad schematic)
At the start: 11 parts, among them J1 Pin_01x05, J2 Pin_01x05, J3 Pin_01x05, J4 Pin_01x05, J5 S5B-PH-SM4-TB

Commit message: Doc tags and PCB_Way files
Other:
- company: (none) -> Dcc DIY Tools
- title: (none) -> DDT I2C Protocol BreakBoard
Changed lines of the file:
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@@
 	(generator_version "8.0")
 	(paper "A4")
+	(title_block
+		(title "DDT I2C Protocol BreakBoard")
+		(date "2024-08-19")
+		(rev "r1")
+		(company "Dcc DIY Tools")
+	)
 	(junction
 		(at 33.02 68.58)
